Commit message: updated Urdf

File: src/ros_unitree/unitree_ros/robots/a1_description/urdf/robot_newton.urdf (robot description, URDF)
Before this commit: robot a1, 33 links, 32 joints
Links:
- removed link camera_color_frame
- removed link camera_color_optical_frame
- removed link camera_depth_frame
- removed link camera_depth_optical_frame
- removed link camera_left_ir_frame
- removed link camera_left_ir_optical_frame
- removed link camera_right_ir_frame
- removed link camera_right_ir_optical_frame
- link camera_link: mass 0.564 -> 0.264
Joints:
- removed joint camera_color_joint
- removed joint camera_color_optical_joint
- removed joint camera_depth_joint
- removed joint camera_depth_optical_joint
- removed joint camera_left_ir_joint
- removed joint camera_left_ir_optical_joint
- removed joint camera_right_ir_joint
- removed joint camera_right_ir_optical_joint
