Commit message: fixed changes for urdfs

File: src/ros_unitree/unitree_ros/robots/a1_description/urdf/robot.urdf (robot description, URDF)
Before this commit: robot a1, 33 links, 32 joints
Links:
- link camera_link: mass 0.564 -> 0.200

File: src/ros_unitree/unitree_ros/robots/a1_description/urdf/robot_newton.urdf (robot description, URDF)
Before this commit: robot a1, 25 links, 24 joints
Links:
- link camera_link: mass 0.264 -> 0.200

File: src/ros_unitree/unitree_ros/robots/a1_description/xacro/_d435.urdf.xacro (robot description, xacro)
@@ -57,6 +57,5 @@
                 <mass value="0.200" />
                 <origin xyz="0 0 0" />
-                <inertia ixx="2.083e-5" ixy="0.0" ixz="0.0" iyy="1.452e-4"" iyz="0.0"
-                    izz="1.452e-4" />
+                <inertia ixx="2.083e-5" ixy="0.0" ixz="0.0" iyy="1.452e-4" iyz="0.0" izz="1.452e-4" />
             </inertial>
         </link>

Commit message: Define inertial properties for camera_bottom_screw_frame
Added inertial properties to the camera_bottom_screw_frame link.

File: src/ros_unitree/unitree_ros/robots/a1_description/urdf/robot.urdf (robot description, URDF)
Before this commit: robot a1, 33 links, 32 joints
Links:
- link camera_bottom_screw_frame: mass None -> 0.001
