Commit message: Update mass and inertia values in URDF Xacro file

File: src/ros_unitree/unitree_ros/robots/a1_description/xacro/_d435.urdf.xacro (robot description, xacro)
@@ -55,8 +55,8 @@
             <inertial>
                 <!-- The following are not reliable values, and should not be used for modeling -->
-                <mass value="0.564" />
+                <mass value="0.200" />
                 <origin xyz="0 0 0" />
-                <inertia ixx="0.003881243" ixy="0.0" ixz="0.0" iyy="0.000498940" iyz="0.0"
-                    izz="0.003879257" />
+                <inertia ixx="2.083e-5" ixy="0.0" ixz="0.0" iyy="1.452e-4"" iyz="0.0"
+                    izz="1.452e-4" />
             </inertial>
         </link>

Commit message: Update _d435.urdf.xacro

File: src/ros_unitree/unitree_ros/robots/a1_description/xacro/_d435.urdf.xacro (robot description, xacro)
@@ -29,5 +29,11 @@
             <child link="${name}_bottom_screw_frame" />
         </joint>
-        <link name="${name}_bottom_screw_frame" />
+        <link name="${name}_bottom_screw_frame">
+            <inertial>
+                <mass value="0.001"/>
+                <origin rpy="0 0 0" xyz="0 0 0"/>
+                <inertia ixx="0.0001" ixy="0" ixz="0" iyy="0.0001" iyz="0" izz="0.0001"/>
+            </inertial>
+        </link>
         <joint name="${name}_link_joint" type="fixed">
             <origin xyz="0 ${d435_cam_depth_py} ${d435_cam_depth_pz}" rpy="0 0 0" />
