Commit message: Refactor laser frame and joint names in URDF

File: src/ros_unitree/unitree_ros/robots/a1_description/xacro/hokuyo_urg04lx.urdf.xacro (robot description, xacro)
@@ -49,11 +49,11 @@
       </gazebo>
     </xacro:macro>
-    <xacro:hokuyo_urg04lx frame="${prefix}_laser" topic="${topic}" />
-    <joint name="${prefix}_laser_mount_joint" type="fixed">
+    <xacro:hokuyo_urg04lx frame="laser" topic="${topic}" />
+    <joint name="${prefix}_laser_base_joint" type="fixed">
       <xacro:insert_block name="origin" />
       <parent link="${parent_link}" />
-      <child link="${prefix}_laser_mount" />
+      <child link="$laser_base" />
     </joint>
-    <link name="${prefix}_laser_mount">
+    <link name="laser_base">
       <visual>
         <origin xyz="0 0 0" rpy="1.57 0 0" />
@@ -72,8 +72,8 @@
     <joint name="${prefix}_laser_joint" type="fixed">
       <origin xyz="0 0 0.064" rpy="0 0 0" />
-      <parent link="${prefix}_laser_mount" />
-      <child link="${prefix}_laser" />
+      <parent link="laser_base" />
+      <child link="laser" />
     </joint>
-    <gazebo reference="${prefix}_laser_mount">
+    <gazebo reference="laser_base">
       <material>Gazebo/DarkGrey</material>
     </gazebo>

Commit message: Fix child link reference in laser base joint

File: src/ros_unitree/unitree_ros/robots/a1_description/xacro/hokuyo_urg04lx.urdf.xacro (robot description, xacro)
@@ -53,5 +53,5 @@
       <xacro:insert_block name="origin" />
       <parent link="${parent_link}" />
-      <child link="$laser_base" />
+      <child link="laser_base" />
     </joint>
     <link name="laser_base">
